Commit message: update stuff

File: src/resources/test_hand/test_hand_non_scale.urdf (robot description, URDF)
Before this commit: robot test_hand, 5 links, 4 joints
Links:
- link finger0_segment0: geometry collision mesh filename=obj_files/finger0_segment0_collision.obj scale=1 1 1; visual mesh filename=obj_files/finger0_segment0.obj scale=1 1 1
- link finger0_segment1: geometry collision mesh filename=obj_files/finger0_segment1_collision.obj scale=1 1 1; visual mesh filename=obj_files/finger0_segment1.obj scale=1 1 1
- link finger1_segment0: geometry collision mesh filename=obj_files/finger1_segment0_collision.obj scale=1 1 1; visual mesh filename=obj_files/finger1_segment0.obj scale=1 1 1
- link finger1_segment1: geometry collision mesh filename=obj_files/finger1_segment1_collision.obj scale=1 1 1; visual mesh filename=obj_files/finger1_segment1.obj scale=1 1 1
- link palm: geometry collision mesh filename=obj_files/palm_collision.obj scale=1 1 1; visual mesh filename=obj_files/palm.obj scale=1 1 1
Joints:
- joint finger0_segment0_joint: axis 1 0 0 -> -1 0 0; origin xyz=0.0 0.075 0 rpy=0 0 0 -> xyz=0.0 0.75 0 rpy=0 0 0
- joint finger0_segment1_joint: origin xyz=0 0 0.06 rpy=0 0 0 -> xyz=0 0 0.6 rpy=0 0 0
- joint finger1_segment0_joint: origin xyz=.9184850993605148e-17 -0.075 0 rpy=0 0 0.0 -> xyz=9.184850993605148e-17 -0.75 0 rpy=0 0 0.0
- joint finger1_segment1_joint: origin xyz=0 0 0.06 rpy=0 0 0 -> xyz=0 0 0.6 rpy=0 0 0
