Commit message: updating code and adding new controller class

File: src/resources/test_hand/test_hand.urdf (robot description, URDF)
Before this commit: robot test_hand, 5 links, 4 joints
Joints:
- joint finger1_segment0_joint: origin xyz=.9184850993605148e-17 -0.075 0 rpy=0 0 0.0 -> xyz=0 -0.075 0 rpy=0 0 0.0
